Commit message: Add workcell scene: pillar, table, conveyor belt with ros2_control

File: src/wm_ur20_description/urdf/ur20_ros2_control.xacro (robot description, xacro)
@@ -48,4 +48,10 @@
         <state_interface name="effort"/>
       </joint>
+      <!-- Conveyor belt slide joint — velocity command, position/velocity state -->
+      <joint name="belt_slide">
+        <command_interface name="velocity"/>
+        <state_interface name="position"><param name="initial_value">0.0</param></state_interface>
+        <state_interface name="velocity"><param name="initial_value">0.0</param></state_interface>
+      </joint>
     </ros2_control>
   </xacro:macro>
