Commit message: Fix: add finger_left_slide dummy URDF joint so mujoco_system registers it
mujoco_ros2_control looks up every ros2_control joint in the URDF before
registering the hardware interface. finger_left_slide only existed in the
MJCF (scene.xacro) — missing from the URDF caused 'Joint not found' warn
and finger_left_slide/position to be listed as 'Not existing', blocking
all controller activation including joint_state_broadcaster.

Same pattern as belt_slide: dummy prismatic link parented to world.

Co-Authored-By: Claude Sonnet 4.6 <noreply@anthropic.com>

File: src/wm_ur20_description/urdf/ur20_mujoco.urdf.xacro (robot description, xacro)
@@ -14,4 +14,12 @@
     <axis xyz="1 0 0"/>
     <limit lower="-100" upper="100" effort="2000" velocity="1.0"/>
+  </joint>
+  <!-- Gripper finger link — dummy link so mujoco_system can find finger_left_slide in the URDF -->
+  <link name="finger_left_link"/>
+  <joint name="finger_left_slide" type="prismatic">
+    <parent link="world"/>
+    <child link="finger_left_link"/>
+    <axis xyz="0 -1 0"/>
+    <limit lower="-0.04" upper="0.04" effort="100" velocity="0.5"/>
   </joint>
   <!-- Instantiate UR20 — generate_ros2_control_tag=false so we supply our own block -->
