Commit message: Phase 5: integrate 2FG14 gripper into scene.xacro pipeline
Mesh housekeeping:
- Move 2FG14_basep2/3.STL and 2FG14_gripper_finger.STL from repo root
  to src/wm_ur20_description/meshes/collision/ where meshdir points
- Remove standalone ur20v2.xml (gripper now lives in scene.xacro)

scene.xacro:
- Add 4 gripper mesh assets and blue_plastic/black_plastic materials
- Add gripper body under wrist_3_link: base parts + finger_left/right
  bodies with slide joints (range -0.04..0.04 m, damping 50)
- Add finger contact exclusions (wrist_3↔gripper, gripper↔fingers)
- Add equality constraint (anti-coupled polycoef="0 -1") for symmetric grasp
- Add 'fingers' position actuator (kp=2000, 0.00245=closed, 0.028=open)
- Fix keyframe to 9 qpos / 8 ctrl values (added two finger DOFs)

ros2_control:
- Add finger_left_slide joint (position cmd, pos/vel state, initial=0.028)
- Add gripper_position_controller (ForwardCommandController, position)
- Spawn gripper_position_controller in launch file alongside arm controllers

Co-Authored-By: Claude Sonnet 4.6 <noreply@anthropic.com>

File: src/wm_cell_description/mjcf/scene.xacro (robot description, xacro)
@@ -64,11 +64,18 @@
     <mesh name="wrist2_vis"   file="visual/wrist2.obj"/>
     <mesh name="wrist3_vis"   file="visual/wrist3.obj"/>
-    <material name="ur_metal"   rgba="0.27 0.27 0.27 1" specular="0.85" shininess="0.75" reflectance="0.10"/>
-    <material name="ur_link"    rgba="0.33 0.33 0.33 1" specular="0.70" shininess="0.60" reflectance="0.05"/>
-    <material name="floor_mat"  rgba="0.45 0.45 0.45 1" specular="0.10" shininess="0.10"/>
-    <material name="pillar_mat" rgba="0.50 0.50 0.55 1" specular="0.60" shininess="0.50"/>
-    <material name="table_mat"  rgba="0.80 0.72 0.58 1" specular="0.30" shininess="0.40"/>
-    <material name="frame_mat"  rgba="0.35 0.35 0.40 1" specular="0.50" shininess="0.40"/>
-    <material name="belt_mat"   rgba="0.12 0.12 0.12 1" specular="0.20" shininess="0.20"/>
+    <!-- OnRobot 2FG14 gripper meshes (collision used for both rendering and contact) -->
+    <mesh name="gripper_base1_col"  file="collision/2FG14_basep1.STL"/>
+    <mesh name="gripper_base2_col"  file="collision/2FG14_basep2.STL"/>
+    <mesh name="gripper_base3_col"  file="collision/2FG14_basep3.STL"/>
+    <mesh name="gripper_finger_col" file="collision/2FG14_gripper_finger.STL"/>
+    <material name="ur_metal"      rgba="0.27 0.27 0.27 1" specular="0.85" shininess="0.75" reflectance="0.10"/>
+    <material name="ur_link"       rgba="0.33 0.33 0.33 1" specular="0.70" shininess="0.60" reflectance="0.05"/>
+    <material name="floor_mat"     rgba="0.45 0.45 0.45 1" specular="0.10" shininess="0.10"/>
+    <material name="pillar_mat"    rgba="0.50 0.50 0.55 1" specular="0.60" shininess="0.50"/>
+    <material name="table_mat"     rgba="0.80 0.72 0.58 1" specular="0.30" shininess="0.40"/>
+    <material name="frame_mat"     rgba="0.35 0.35 0.40 1" specular="0.50" shininess="0.40"/>
+    <material name="belt_mat"      rgba="0.12 0.12 0.12 1" specular="0.20" shininess="0.20"/>
+    <material name="blue_plastic"  rgba="0.10 0.10 0.80 1" specular="0.10" shininess="0.10"/>
+    <material name="black_plastic" rgba="0.10 0.10 0.10 1" specular="0.10" shininess="0.10"/>
   </asset>
   <contact>
@@ -79,4 +86,7 @@
     <exclude body1="wrist_1_link"   body2="wrist_2_link"/>
     <exclude body1="wrist_2_link"   body2="wrist_3_link"/>
+    <exclude body1="wrist_3_link"   body2="gripper"/>
+    <exclude body1="gripper"        body2="finger_left"/>
+    <exclude body1="gripper"        body2="finger_right"/>
   </contact>
   <worldbody>
@@ -148,4 +158,44 @@
                 <geom name="wrist3_col" pos="0 0 -0.07" quat="0.707107 0.707107 0 0" type="mesh" mesh="wrist3_col" group="3" contype="1" conaffinity="1"/>
                 <site name="ee_site" pos="0 0 0" size="0.01" rgba="1 0 0 1"/>
+                <!-- ════════════════════════════════════════
+                     OnRobot 2FG14 GRIPPER
+                     Attached to wrist_3_link.
+                     One actuator drives finger_left_slide; equality couples finger_right.
+                     ctrl range: 0.00245 m (closed) → 0.028 m (fully open).
+                     To open:  pub 0.028 to /gripper_position_controller/commands
+                     To close: pub 0.00245 to /gripper_position_controller/commands
+                     ════════════════════════════════════════ -->
+                <body name="gripper" pos="0 0 0" quat="1 0 0 0">
+                  <geom name="gripper_base1" pos="0 0 0" quat="1 0 0 0"
+                        type="mesh" mesh="gripper_base1_col"
+                        group="0" material="blue_plastic"
+                        contype="1" conaffinity="1" density="2200"/>
+                  <geom name="gripper_base2" pos="0 0 0.013" quat="1 0 0 0"
+                        type="mesh" mesh="gripper_base2_col"
+                        group="0" material="ur_metal"
+                        contype="1" conaffinity="1" density="5000"/>
+                  <geom name="gripper_base3" pos="0 0 0.103" quat="0.707107 0 0 0.707107"
+                        type="mesh" mesh="gripper_base3_col"
+                        group="0" material="black_plastic"
+                        contype="1" conaffinity="1" density="5000"/>
+                  <body name="finger_left" pos="0 -0.0025 0.1137" quat="1 0 0 0">
+                    <joint name="finger_left_slide" type="slide" pos="0 0 0" axis="0 -1 0"
+                           range="-0.04 0.04" damping="50"/>
+                    <geom name="finger_left_col" pos="0 0 0" quat="1 0 0 0"
+                          type="mesh" mesh="gripper_finger_col"
+                          group="0" material="blue_plastic"
+                          friction="1.5 0.05 0.01" contype="1" conaffinity="1" density="5000"/>
+                    <site name="finger_left_tip" pos="0 0 0.069" size="0.005" rgba="1 0 0 1"/>
+                  </body>
+                  <body name="finger_right" pos="0 0.0025 0.1137" quat="0 0 0 1">
+                    <joint name="finger_right_slide" type="slide" pos="0 0 0" axis="0 -1 0"
+                           range="-0.04 0.04" damping="50"/>
+                    <geom name="finger_right_col" pos="0 0 0" quat="1 0 0 0"
+                          type="mesh" mesh="gripper_finger_col"
+                          group="0" material="blue_plastic"
+                          friction="1.5 0.05 0.01" contype="1" conaffinity="1" density="5000"/>
+                    <site name="finger_right_tip" pos="0 0 0.069" size="0.005" rgba="0 1 0 1"/>
+                  </body>
+                </body>
               </body>
             </body>
@@ -233,8 +283,23 @@
     <!-- Belt: velocity-controlled (m/s).  +X = forward toward human station. -->
     <velocity name="belt_motor" joint="belt_slide" kv="2000" ctrlrange="-1.0 1.0"/>
+    <!-- Gripper: position-controlled. Drives finger_left_slide; equality couples finger_right.
+         0.00245 m = closed,  0.028 m = fully open -->
+    <position name="fingers" joint="finger_left_slide" kp="2000" ctrlrange="0.00245 0.028"/>
   </actuator>
-  <!-- 7 values: 6 arm joints + belt_slide (0 = parked at start) -->
+  <!-- Equality: couple both finger slides so one actuator opens/closes symmetrically.
+       polycoef="0 -1 ..." means finger_right = -finger_left (anti-coupled → symmetric grasp) -->
+  <equality>
+    <joint name="fingers_eq"
+           joint1="finger_left_slide" joint2="finger_right_slide"
+           polycoef="0 -1 0 0 0"
+           solref="0.02 1" solimp="0.9 0.95 0.001"/>
+  </equality>
+  <!-- qpos order (depth-first): 6 arm joints, finger_left, finger_right, belt_slide = 9 values
+       ctrl  order (actuator):   6 arm,        belt_motor,  fingers               = 8 values
+       Gripper starts open (0.028 m); belt parked (0). -->
   <keyframe>
-    <key name="home" qpos="0 -1.5708 0 0 0 0 0" ctrl="0 -1.5708 0 0 0 0 0"/>
+    <key name="home"
+         qpos="0 -1.5708 0 0 0 0  0.028 -0.028  0"
+         ctrl="0 -1.5708 0 0 0 0  0  0.028"/>
   </keyframe>
 </mujoco>

File: src/wm_ur20_description/urdf/ur20_ros2_control.xacro (robot description, xacro)
@@ -54,4 +54,10 @@
         <state_interface name="velocity"><param name="initial_value">0.0</param></state_interface>
       </joint>
+      <!-- 2FG14 gripper — position command on left finger; equality in MJCF drives right -->
+      <joint name="finger_left_slide">
+        <command_interface name="position"/>
+        <state_interface name="position"><param name="initial_value">0.028</param></state_interface>
+        <state_interface name="velocity"><param name="initial_value">0.0</param></state_interface>
+      </joint>
     </ros2_control>
   </xacro:macro>

Commit message: Phase 6: assembly state machine + drum-cap workpiece
- wm_assembly_ctrl/assembly_node.py: 12-state timer-driven pick-and-place
  (IDLE→STAGING→SETTLING→PRE_PICK→DESCEND→GRASPING→LIFTING→
   TRANSITING→PLACING→RELEASING→RETRACTING→HOMING→DONE).
  Belt stages drum cap from x=−0.9 to x≈0, IK node handles arm motion,
  gripper controller handles grasp/release.

- scene.xacro: add red 50mm cylinder drum_cap as free body on belt,
  drum_cap_mat material, keyframe extended to 16 qpos (adds freejoint 7-vec).

- ur20_mujoco.launch.py: assembly_node spawns at t=12 s, guarded by
  launch arg assembly:=false (opt-in). Add assembly DeclareLaunchArgument.

- wm_assembly_ctrl setup.py / package.xml: wire assembly_node entry point,
  add std_msgs dependency.

Co-Authored-By: Claude Sonnet 4.6 <noreply@anthropic.com>

File: src/wm_cell_description/mjcf/scene.xacro (robot description, xacro)
@@ -78,4 +78,5 @@
     <material name="blue_plastic"  rgba="0.10 0.10 0.80 1" specular="0.10" shininess="0.10"/>
     <material name="black_plastic" rgba="0.10 0.10 0.10 1" specular="0.10" shininess="0.10"/>
+    <material name="drum_cap_mat"  rgba="0.85 0.15 0.15 1" specular="0.20" shininess="0.30"/>
   </asset>
   <contact>
@@ -279,4 +280,17 @@
             contype="1" conaffinity="1"/>
     </body>
+    <!-- ════════════════════════════════════════
+         ASSEMBLY PART — washing-machine drum top cap
+         Starts at x = −0.9 m on the belt; Phase 6 state machine runs the belt
+         for 3 s at +0.3 m/s to slide it to x ≈ 0 (pick site), then stops.
+         diameter = 50 mm, height = 40 mm — grippable by the 2FG14 (range 24–75 mm).
+         ════════════════════════════════════════ -->
+    <body name="drum_cap" pos="-0.9 ${conv_cy} ${conv_h + 0.020}">
+      <freejoint/>
+      <geom name="drum_cap_geom" type="cylinder" size="0.025 0.020"
+            mass="2.0" material="drum_cap_mat"
+            friction="0.8 0.05 0.01" condim="4"
+            contype="1" conaffinity="1"/>
+    </body>
   </worldbody>
   <!-- ════════════════════════════════════════
@@ -306,10 +320,11 @@
            solref="0.02 1" solimp="0.9 0.95 0.001"/>
   </equality>
-  <!-- qpos order (depth-first): 6 arm joints, finger_left, finger_right, belt_slide = 9 values
+  <!-- qpos order (depth-first): 6 arm joints, finger_left, finger_right, belt_slide,
+                                  drum_cap freejoint (x y z qw qx qy qz) = 16 values
        ctrl  order (actuator):   6 arm,        belt_motor,  fingers               = 8 values
-       Gripper starts open (0.028 m); belt parked (0). -->
+       Gripper starts open (0.028 m); belt parked (0); drum_cap at pick-staging site. -->
   <keyframe>
     <key name="home"
-         qpos="0 -1.5708 0 0 0 0  0.028 0.028  0"
+         qpos="0 -1.5708 0 0 0 0  0.028 0.028  0  -0.9 -0.9 0.52 1 0 0 0"
          ctrl="0 -1.5708 0 0 0 0  0  0.028"/>
   </keyframe>
